File: Fence/fencerSMD.brd (EAGLE design)
At the start: 101.3 x 27.9 mm, 35 parts, among them IC1 NE555D, IC5 NE555D, IC6 NE555D, Q1 IRF640N-H, X1 12V

Commit message: Updating stuff that was not before
Parts:
- Q1: value IRF640N-H -> IRF640NS; device IRF640:TO220 -> IRF640:D2PAK
- moved X2 10.2 mm to (99.1, 38.1)
- moved X1 4.58 mm to (94.0, 50.8)
- moved PULSES 1.80 mm to (73.7, 38.1), turned to 270 degrees
- moved Q1 1.80 mm to (87.6, 38.1)
Routing:
- net EARTHGROUND: track 24.0 -> 9.95 mm
- net ACC: track 14.7 -> 19.3 mm
- net N$6: track 5.14 -> 2.25 mm
- net T1: track 22.1 -> 23.1 mm
- net N$8: track 5.45 -> 6.30 mm
