File: Fence/fencerSMD.sch (EAGLE design)
At the start: 35 parts, among them IC1 NE555D, IC5 NE555D, IC6 NE555D, Q1 IRF640N-H, X1 12V

Commit message: Updating stuff that was not before
Parts:
- Q1: value IRF640N-H -> IRF640NS; device IRF640:IRF640N-H -> IRF640:IRF640NS
Changed lines of the file:
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@@
 <part name="PULSES" library="fab (1)" deviceset="LED" device="FAB1206" value="Blue"/>
 <part name="GND13" library="01_FAB_Hello" deviceset="GND" device=""/>
-<part name="Q1" library="IRF640" deviceset="IRF640" device="N-H"/>
+<part name="Q1" library="IRF640" deviceset="IRF640" device="NS" value="IRF640NS"/>
 <part name="GND14" library="01_FAB_Hello" deviceset="GND" device=""/>
 <part name="R12" library="01_FAB_Hello" deviceset="RESISTOR" device="1206" value="0"/>
