File: Fence2/electric_fence.brd (EAGLE design)
At the start: 100 x 80 mm, 34 parts, among them IC1 LM555D, IC2 LM555D, IC3 LM555D, Q1 IRF3704S

Commit message: 1
Parts:
- moved C10 75.5 mm to (87.6, 66.0), turned to 180 degrees
- turned C8 to 180 degrees
- turned LED3 to 270 degrees
- turned R10 to 270 degrees
- turned R11 to 90 degrees
- turned R9 to 180 degrees
Routing:
- net N$15: track 0.00 -> 203.0 mm
- net N$22: track 0.00 -> 86.7 mm
- net +12V: track 0.00 -> 84.5 mm
- net N$5: track 0.00 -> 79.3 mm
- net N$16: track 0.00 -> 42.7 mm
- net N$7: track 0.00 -> 36.8 mm
- net N$9: track 0.00 -> 33.7 mm
- net N$4: track 0.00 -> 33.5 mm
- net N$12: track 0.00 -> 31.1 mm
- net N$13: track 0.00 -> 27.8 mm
- net N$6: track 0.00 -> 25.3 mm
- net N$23: track 0.00 -> 23.7 mm
- net N$11: track 0.00 -> 21.1 mm
- net N$10: track 0.00 -> 19.9 mm
- net N$18: track 0.00 -> 16.0 mm
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- added copper zone on layer 1, net GND
